Commit message: Add base_link & additional two joints
This commit adds a base link which keeps the model from breaking
apart when we launch gazebo.
Additionally two elbow/forearm joints are renamed / correctly added.

Joints have been changed from continuous to revolute with upper/lower
limits taken from provided documentation (Compliant Bimanual ...).

Corrections for the rotation axis for each joint are implemented as
well.

File: antrop_arms_description/urdf/antrop_arms.xacro (robot description, xacro)
@@ -4,4 +4,5 @@
 <xacro:include filename="$(find antrop_arms_description)/urdf/antrop_arms.trans" />
 <xacro:include filename="$(find antrop_arms_description)/urdf/antrop_arms.gazebo" />
+<link name="world"/>
 <link name="base_link">
   <inertial>
@@ -264,9 +265,11 @@
   </collision>
 </link>
-<joint name="base_shoulder_left_joint" type="continuous">
+<joint name="base_shoulder_left_joint" type="revolute">
   <origin xyz="0.021 0.04 -0.0" rpy="0 0 0"/>
   <parent link="shoulder_left_link_1"/>
   <child link="Shoulder_Yaw_Structure_v1_1"/>
   <axis xyz="1.0 -0.0 0.0"/>
+  <limit effort="20.1" velocity="2" lower="-0.174533" upper="1.5708" />
+  <!--Here we should keep in mind exactly which arm we are looking at since the limits are opposite when it comes to upper/lower limit for each side-->
 </joint>
 <joint name="Rigid3" type="fixed">
@@ -280,15 +283,18 @@
   <child link="Shoulder_Yaw_Transmission_v1_1"/>
 </joint>
-<joint name="shoulder_elbow_left_joint" type="continuous">
+<joint name="shoulder_elbow_left_joint" type="revolute">
   <origin xyz="0.0 0.0 -0.048" rpy="0 0 0"/>
   <parent link="Shoulder_Yaw_Transmission_v1_1"/>
   <child link="elbow_left_link_1"/>
   <axis xyz="0.0 0.0 1.0"/>
-</joint>
-<joint name="base_shoulder_right_joint" type="continuous">
+  <limit effort="20.1" velocity="2" lower="-1.5708" upper="1.5708" />
+</joint>
+<joint name="base_shoulder_right_joint" type="revolute">
   <origin xyz="0.021 -0.04 -0.0" rpy="0 0 0"/>
   <parent link="shoulder_right_link_1"/>
   <child link="Shoulder_Yaw_Structure_v1__1__1"/>
-  <axis xyz="1.0 -0.0 0.0"/>
+  <axis xyz="1 0 0" />
+  <limit effort="20.1" velocity="2" lower="-1.5708" upper="0.174533" /><!--"0.174533" corresponds to 10 degrees transformed to radians-->
+  <!--Here we should keep in mind exactly which arm we are looking at since the limits are opposite when it comes to upper/lower limit for each side-->
 </joint>
 <joint name="Rigid9" type="fixed">
@@ -302,9 +308,10 @@
   <child link="Shoulder_Yaw_Transmission_v1__1__1"/>
 </joint>
-<joint name="shoulder_elbow_right_joint" type="continuous">
+<joint name="shoulder_elbow_right_joint" type="revolute">
   <origin xyz="0.0 0.0 -0.048" rpy="0 0 0"/>
   <parent link="Shoulder_Yaw_Transmission_v1__1__1"/>
   <child link="elbow_right_link_1"/>
   <axis xyz="0.0 -0.0 1.0"/>
+  <limit effort="20.1" velocity="2" lower="-1.5708" upper="1.5708" />
 </joint>
 <joint name="base_shoulder_right_fixed_joint" type="fixed">
@@ -318,13 +325,22 @@
   <child link="shoulder_left_link_1"/>
 </joint>
-<joint name="Rigid17" type="fixed">
+<joint name="elbow_forearm_right_joint" type="revolute">
   <origin xyz="0.0 0.02 -0.1395" rpy="0 0 0"/>
+  <limit effort="20.1" velocity="2" lower="-2.35619" upper="2.35619" />
+  <axis xyz="0 1 0" />
   <parent link="elbow_right_link_1"/>
+  <child link="forearm_right_link_1"/>
+</joint>
+<joint name="elbow_forearm_left_joint" type="revolute">
+  <origin xyz="0.0 0.02 -0.1395" rpy="0 0 0"/>
+  <limit effort="20.1" velocity="2" lower="-2.35619" upper="2.35619" />
+  <parent link="elbow_left_link_1"/>
+  <axis xyz="0 1 0" />
   <child link="forearm_left_link_1"/>
 </joint>
-<joint name="Rigid18" type="fixed">
-  <origin xyz="0.0 0.02 -0.1395" rpy="0 0 0"/>
-  <parent link="elbow_left_link_1"/>
-  <child link="forearm_right_link_1"/>
+<joint name="float_base_link" type="fixed">
+  <origin xyz="0 0 1.5" rpy="0 0 0"/>
+  <parent link="world"/>
+  <child link="base_link"/>
 </joint>
 </robot>

Commit message: Add shoulder pitch joint
This commit adds an additional axis of rotation.
Precisely the shoulder pitch for both arms which
was missing and causing issues when simulating.

Additionally this commit adds a more clear urdf
layout with more comments for easier understanding.

File: antrop_arms_description/urdf/antrop_arms.xacro (robot description, xacro)
@@ -4,5 +4,9 @@
 <xacro:include filename="$(find antrop_arms_description)/urdf/antrop_arms.trans" />
 <xacro:include filename="$(find antrop_arms_description)/urdf/antrop_arms.gazebo" />
+<!--Virtual links only used for simulation work-->
 <link name="world"/>
+<link name="right_ee_link"/>
+<link name="left_ee_link"/>
+<!--Actual robot links-->
 <link name="base_link">
   <inertial>
@@ -25,4 +29,6 @@
   </collision>
 </link>
+<!--Left side of the robot-->
+<!--Left shoulder-->
 <link name="Shoulder_Yaw_Structure_v1_1">
   <inertial>
@@ -85,4 +91,25 @@
   </collision>
 </link>
+<link name="shoulder_left_link_1">
+  <inertial>
+    <origin xyz="-0.0002500317321533693 0.035918090920304124 -0.013543028885077059" rpy="0 0 0"/>
+    <mass value="0.6591423872621155"/>
+    <inertia ixx="0.000324" iyy="0.000242" izz="0.000235" ixy="-9e-06" iyz="3.6e-05" ixz="2e-06"/>
+  </inertial>
+  <visual>
+    <origin xyz="0.0 -0.14 -0.0" rpy="0 0 0"/>
+    <geometry>
+      <mesh filename="package://antrop_arms_description/meshes/shoulder_left_link_1.stl" scale="0.001 0.001 0.001"/>
+    </geometry>
+    <material name="silver"/>
+  </visual>
+  <collision>
+    <origin xyz="0.0 -0.14 -0.0" rpy="0 0 0"/>
+    <geometry>
+      <mesh filename="package://antrop_arms_description/meshes/shoulder_left_link_1.stl" scale="0.001 0.001 0.001"/>
+    </geometry>
+  </collision>
+</link>
+<!--Left elbow-->
 <link name="elbow_left_link_1">
   <inertial>
@@ -105,4 +132,27 @@
   </collision>
 </link>
+<!--Left forearm-->
+<link name="forearm_left_link_1">
+  <inertial>
+    <origin xyz="-2.4015511801422917e-14 -0.020000000000116203 -0.14499270392199487" rpy="0 0 0"/>
+    <mass value="0.20799291557495453"/>
+    <inertia ixx="0.001901" iyy="0.001879" izz="3.1e-05" ixy="-0.0" iyz="0.0" ixz="-0.0"/>
+  </inertial>
+  <visual>
+    <origin xyz="0.0155 0.16 0.3025" rpy="0 0 0"/>
+    <geometry>
+      <mesh filename="package://antrop_arms_description/meshes/forearm_left_link_1.stl" scale="0.001 0.001 0.001"/>
+    </geometry>
+    <material name="silver"/>
+  </visual>
+  <collision>
+    <origin xyz="0.0155 0.16 0.3025" rpy="0 0 0"/>
+    <geometry>
+      <mesh filename="package://antrop_arms_description/meshes/forearm_left_link_1.stl" scale="0.001 0.001 0.001"/>
+    </geometry>
+  </collision>
+</link>
+<!--Right side of the robot-->
+<!--Right shoulder-->
 <link name="Shoulder_Yaw_Structure_v1__1__1">
   <inertial>
@@ -165,4 +215,25 @@
   </collision>
 </link>
+<link name="shoulder_right_link_1">
+  <inertial>
+    <origin xyz="-0.0002500317321433487 -0.03591809092030432 -0.013543028885077014" rpy="0 0 0"/>
+    <mass value="0.6591423872621155"/>
+    <inertia ixx="0.000324" iyy="0.000242" izz="0.000235" ixy="9e-06" iyz="-3.6e-05" ixz="2e-06"/>
+  </inertial>
+  <visual>
+    <origin xyz="0.0 0.14 -0.0" rpy="0 0 0"/>
+    <geometry>
+      <mesh filename="package://antrop_arms_description/meshes/shoulder_right_link_1.stl" scale="0.001 0.001 0.001"/>
+    </geometry>
+    <material name="silver"/>
+  </visual>
+  <collision>
+    <origin xyz="0.0 0.14 -0.0" rpy="0 0 0"/>
+    <geometry>
+      <mesh filename="package://antrop_arms_description/meshes/shoulder_right_link_1.stl" scale="0.001 0.001 0.001"/>
+    </geometry>
+  </collision>
+</link>
+<!--Right elbow-->
 <link name="elbow_right_link_1">
   <inertial>
@@ -185,64 +256,5 @@
   </collision>
 </link>
-<link name="shoulder_right_link_1">
-  <inertial>
-    <origin xyz="-0.0002500317321433487 -0.03591809092030432 -0.013543028885077014" rpy="0 0 0"/>
-    <mass value="0.6591423872621155"/>
-    <inertia ixx="0.000324" iyy="0.000242" izz="0.000235" ixy="9e-06" iyz="-3.6e-05" ixz="2e-06"/>
-  </inertial>
-  <visual>
-    <origin xyz="0.0 0.14 -0.0" rpy="0 0 0"/>
-    <geometry>
-      <mesh filename="package://antrop_arms_description/meshes/shoulder_right_link_1.stl" scale="0.001 0.001 0.001"/>
-    </geometry>
-    <material name="silver"/>
-  </visual>
-  <collision>
-    <origin xyz="0.0 0.14 -0.0" rpy="0 0 0"/>
-    <geometry>
-      <mesh filename="package://antrop_arms_description/meshes/shoulder_right_link_1.stl" scale="0.001 0.001 0.001"/>
-    </geometry>
-  </collision>
-</link>
-<link name="shoulder_left_link_1">
-  <inertial>
-    <origin xyz="-0.0002500317321533693 0.035918090920304124 -0.013543028885077059" rpy="0 0 0"/>
-    <mass value="0.6591423872621155"/>
-    <inertia ixx="0.000324" iyy="0.000242" izz="0.000235" ixy="-9e-06" iyz="3.6e-05" ixz="2e-06"/>
-  </inertial>
-  <visual>
-    <origin xyz="0.0 -0.14 -0.0" rpy="0 0 0"/>
-    <geometry>
-      <mesh filename="package://antrop_arms_description/meshes/shoulder_left_link_1.stl" scale="0.001 0.001 0.001"/>
-    </geometry>
-    <material name="silver"/>
-  </visual>
-  <collision>
-    <origin xyz="0.0 -0.14 -0.0" rpy="0 0 0"/>
-    <geometry>
-      <mesh filename="package://antrop_arms_description/meshes/shoulder_left_link_1.stl" scale="0.001 0.001 0.001"/>
-    </geometry>
-  </collision>
-</link>
-<link name="forearm_left_link_1">
-  <inertial>
-    <origin xyz="-2.4015511801422917e-14 -0.020000000000116203 -0.14499270392199487" rpy="0 0 0"/>
-    <mass value="0.20799291557495453"/>
-    <inertia ixx="0.001901" iyy="0.001879" izz="3.1e-05" ixy="-0.0" iyz="0.0" ixz="-0.0"/>
-  </inertial>
-  <visual>
-    <origin xyz="0.0155 0.16 0.3025" rpy="0 0 0"/>
-    <geometry>
-      <mesh filename="package://antrop_arms_description/meshes/forearm_left_link_1.stl" scale="0.001 0.001 0.001"/>
-    </geometry>
-    <material name="silver"/>
-  </visual>
-  <collision>
-    <origin xyz="0.0155 0.16 0.3025" rpy="0 0 0"/>
-    <geometry>
-      <mesh filename="package://antrop_arms_description/meshes/forearm_left_link_1.stl" scale="0.001 0.001 0.001"/>
-    </geometry>
-  </collision>
-</link>
+<!--Right forearm-->
 <link name="forearm_right_link_1">
   <inertial>
@@ -265,4 +277,5 @@
   </collision>
 </link>
+<!--Robot joints-->
 <joint name="base_shoulder_left_joint" type="revolute">
   <origin xyz="0.021 0.04 -0.0" rpy="0 0 0"/>
@@ -315,11 +328,15 @@
   <limit effort="20.1" velocity="2" lower="-1.5708" upper="1.5708" />
 </joint>
-<joint name="base_shoulder_right_fixed_joint" type="fixed">
+<joint name="base_shoulder_right_pitch_joint" type="revolute">
   <origin xyz="0.0 -0.14 0.0" rpy="0 0 0"/>
+  <limit effort="20.1" velocity="2" lower="-1.5708" upper="1.5708" />
+  <axis xyz="0 1 0" />
   <parent link="base_link"/>
   <child link="shoulder_right_link_1"/>
 </joint>
-<joint name="base_shoulder_left_fixed_joint" type="fixed">
+<joint name="base_shoulder_left_pitch_joint" type="revolute">
   <origin xyz="0.0 0.14 0.0" rpy="0 0 0"/>
+  <limit effort="20.1" velocity="2" lower="-1.5708" upper="1.5708" />
+  <axis xyz="0 1 0" />
   <parent link="base_link"/>
   <child link="shoulder_left_link_1"/>
@@ -344,3 +361,13 @@
   <child link="base_link"/>
 </joint>
+<joint name="right_ee" type="fixed">
+  <origin xyz="0 0 -0.225" rpy="0 0 0"/>
+  <parent link="forearm_right_link_1"/>
+  <child link="right_ee_link"/>
+</joint>
+<joint name="left_ee" type="fixed">
+  <origin xyz="0 0 -0.24" ryp="0 0 0"/>
+  <parent link="forearm_left_link_1"/>
+  <child link="left_ee_link"/>
+</joint>
 </robot>
