Commit message: Add entire Moveit_Assistant change

File: antrop_arms_moveit_config/config/gazebo_antrop_arms.urdf (robot description, URDF)
Before this commit: robot antrop_arms, 14 links, 13 joints
Joints:
- joint base_shoulder_left_joint: limit lower=-1.5708 upper=1.5708 effort=20.1 velocity=2 -> lower=-0.174533 upper=1.5708 effort=20.1 velocity=2
- joint base_shoulder_right_joint: limit lower=-1.5708 upper=1.5708 effort=20.1 velocity=2 -> lower=-1.5708 upper=0.174533 effort=20.1 velocity=2

Commit message: Change moveit_config after adding additional joints

File: antrop_arms_moveit_config/config/gazebo_antrop_arms.urdf (robot description, URDF)
Before this commit: robot antrop_arms, 14 links, 13 joints
Links:
- added link left_ee_link
- added link right_ee_link
Joints:
- removed joint base_shoulder_left_fixed_joint
- removed joint base_shoulder_right_fixed_joint
- added joint base_shoulder_left_pitch_joint: type revolute, parent base_link, child shoulder_left_link_1, origin xyz=0.0 0.14 0.0 rpy=0 0 0, axis 0 1 0, limit lower=-1.5708 upper=1.5708 effort=20.1 velocity=2
- added joint base_shoulder_right_pitch_joint: type revolute, parent base_link, child shoulder_right_link_1, origin xyz=0.0 -0.14 0.0 rpy=0 0 0, axis 0 1 0, limit lower=-1.5708 upper=1.5708 effort=20.1 velocity=2
- added joint left_ee: type fixed, parent forearm_left_link_1, child left_ee_link, origin xyz=0 0 -0.24
- added joint right_ee: type fixed, parent forearm_right_link_1, child right_ee_link, origin xyz=0 0 -0.225 rpy=0 0 0
